File: vertical/TOFEAdapter.kicad_pcb (KiCad board)
At the start: 2 copper layers, 51.2 x 24.8 mm, 2 parts, among them U1 TOFE-8X, U2 TOFE-8X

Commit message: Fixing the naming a little.
Parts:
- U1: footprint Inverse:TOFE_8X_Pins -> TOFE Straddle:TOFE_8X_straddle
Changed lines of the file:
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@@
     (links 332)
     (no_connects 3)
-    (area 0 0 0 0)
+    (area 144.431 74.51882 200.010801 103.45898)
     (thickness 1.6)
     (drawings 12)
@@
     (pad "" smd rect (at -1.92618 -13.25088) (size 4 1) (layers F.Cu))
   )
-  (module Inverse:TOFE_8X_Pins (layer B.Cu)
+  (module "TOFE Straddle:TOFE_8X_straddle" (layer B.Cu)
     (at 148.50958 76.69052)
     (fp_text reference U1 (at 0.98044 -0.9271) (layer B.SilkS)
